Commit message: add motor cmd lag

File: legged_gym/resources/robots/go1/urdf/go1.urdf (robot description, URDF)
Before this commit: robot go1_description, 23 links, 22 joints
Links:
- removed link FL_thigh_shoulder
- removed link FR_thigh_shoulder
- removed link RL_thigh_shoulder
- removed link RR_thigh_shoulder
- removed link imu_link
- removed link trunk
- added link imu, mass 0.01; visual box size=0.015 0.015 0.004
- link FL_calf: mass 0.158015 -> 0.135862
- link FL_hip: mass 0.510299 -> 0.591
- link FL_thigh: mass 0.898919 -> 0.92
- link FR_calf: mass 0.158015 -> 0.135862
- link FR_hip: mass 0.510299 -> 0.591
- link FR_thigh: mass 0.898919 -> 0.92
- link RL_calf: mass 0.158015 -> 0.135862
- link RL_hip: mass 0.510299 -> 0.591
- link RL_thigh: mass 0.898919 -> 0.92
- link RR_calf: mass 0.158015 -> 0.135862
- link RR_hip: mass 0.510299 -> 0.591; geometry visual mesh filename=../meshes/hip.stl scale=1 1 1
- link RR_thigh: mass 0.898919 -> 0.92
- link base: mass None -> 5.204; geometry collision box size=0.3762 0.0935 0.114; visual mesh filename=../meshes/trunk.stl scale=1 1 1
Joints:
- removed joint FL_hip_fixed
- removed joint FR_hip_fixed
- removed joint RL_hip_fixed
- removed joint RR_hip_fixed
- removed joint floating_base
- joint FL_calf_joint: limit lower=-2.69653369433 upper=-0.916297857297 effort=33.5 velocity=28 -> lower=-2.818 upper=-0.888 effort=35.55 velocity=20.06
- joint FL_hip_joint: limit lower=-0.802851455917 upper=0.802851455917 effort=33.5 velocity=50 -> lower=-0.863 upper=0.863 effort=23.7 velocity=30.1; parent trunk -> base
- joint FL_thigh_joint: limit lower=-1.0471975512 upper=4.18879020479 effort=33.5 velocity=28 -> lower=-0.686 upper=4.501 effort=23.7 velocity=30.1
- joint FR_calf_joint: limit lower=-2.69653369433 upper=-0.916297857297 effort=33.5 velocity=28 -> lower=-2.818 upper=-0.888 effort=35.55 velocity=20.06
- joint FR_hip_joint: limit lower=-0.802851455917 upper=0.802851455917 effort=33.5 velocity=50 -> lower=-0.863 upper=0.863 effort=23.7 velocity=30.1; parent trunk -> base
- joint FR_thigh_joint: limit lower=-1.0471975512 upper=4.18879020479 effort=33.5 velocity=28 -> lower=-0.686 upper=4.501 effort=23.7 velocity=30.1
- joint RL_calf_joint: limit lower=-2.69653369433 upper=-0.916297857297 effort=33.5 velocity=28 -> lower=-2.818 upper=-0.888 effort=35.55 velocity=20.06
- joint RL_hip_joint: limit lower=-0.802851455917 upper=0.802851455917 effort=33.5 velocity=50 -> lower=-0.863 upper=0.863 effort=23.7 velocity=30.1; parent trunk -> base
- joint RL_thigh_joint: limit lower=-1.0471975512 upper=4.18879020479 effort=33.5 velocity=28 -> lower=-0.686 upper=4.501 effort=23.7 velocity=30.1
- joint RR_calf_joint: limit lower=-2.69653369433 upper=-0.916297857297 effort=33.5 velocity=28 -> lower=-2.818 upper=-0.888 effort=35.55 velocity=20.06
- joint RR_hip_joint: limit lower=-0.802851455917 upper=0.802851455917 effort=33.5 velocity=50 -> lower=-0.863 upper=0.863 effort=23.7 velocity=30.1; parent trunk -> base
- joint RR_thigh_joint: limit lower=-1.0471975512 upper=4.18879020479 effort=33.5 velocity=28 -> lower=-0.686 upper=4.501 effort=23.7 velocity=30.1
- joint imu_joint: child imu_link -> imu; origin xyz=-0.01592 -0.06659 -0.00617 rpy=0 0 0 -> xyz=0. 0. 0. rpy=0. 0. 0.; parent trunk -> base
